File: SensorPCB/SensorPCB.brd (EAGLE design)
At the start: 37 x 65 mm, 31 parts, among them T1 33u

Commit message: update
Parts:
- moved C1 1.28 mm to (2.86, 5.08)
- moved JP1 0.32 mm to (6.51, 3.81)
Routing:
- net +5V: track 15.5 -> 16.8 mm
Other:
- outline, holes or cut-outs redrawn
Changed lines of the file:
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@@
 <layer number="25" name="tNames" color="7" fill="1" visible="yes" active="yes"/>
 <layer number="26" name="bNames" color="7" fill="1" visible="yes" active="yes"/>
-<layer number="27" name="tValues" color="7" fill="1" visible="yes" active="yes"/>
-<layer number="28" name="bValues" color="7" fill="1" visible="yes" active="yes"/>
+<layer number="27" name="tValues" color="7" fill="1" visible="no" active="yes"/>
+<layer number="28" name="bValues" color="7" fill="1" visible="no" active="yes"/>
 <layer number="29" name="tStop" color="7" fill="3" visible="yes" active="yes"/>
 <layer number="30" name="bStop" color="7" fill="6" visible="yes" active="yes"/>
@@
 <layer number="125" name="_tNames" color="7" fill="1" visible="yes" active="yes"/>
 <layer number="126" name="_bNames" color="7" fill="1" visible="yes" active="yes"/>
-<layer number="127" name="_tValues" color="7" fill="1" visible="yes" active="yes"/>
-<layer number="128" name="_bValues" color="7" fill="1" visible="yes" active="yes"/>
+<layer number="127" name="_tValues" color="7" fill="1" visible="no" active="yes"/>
+<layer number="128" name="_bValues" color="7" fill="1" visible="no" active="yes"/>
 <layer number="129" name="Mask" color="7" fill="1" visible="yes" active="yes"/>
 <layer number="131" name="tAdjust" color="7" fill="1" visible="yes" active="yes"/>
@@
 <board>
 <plain>
-<wire x1="0" y1="0" x2="37" y2="0" width="0" layer="20"/>
-<wire x1="37" y1="0" x2="37" y2="65" width="0" layer="20"/>
-<wire x1="37" y1="65" x2="0" y2="65" width="0" layer="20"/>
-<wire x1="0" y1="65" x2="0" y2="0" width="0" layer="20"/>
-<dimension x1="0" y1="0" x2="37" y2="0" x3="18.5" y3="-10" textsize="1.778" layer="1"/>
-<dimension x1="37" y1="0" x2="37" y2="65" x3="58.7375" y3="32.5" textsize="1.778" layer="1"/>
-<text x="6.19125" y="1.905" size="1.27" layer="25" rot="R180">+5V</text>
-<text x="9.8425" y="6.35" size="1.27" layer="25" rot="R180">GND</text>
+<wire x1="2.54" y1="0" x2="34.46" y2="0" width="0" layer="20"/>
+<wire x1="34.46" y1="0" x2="37" y2="2.54" width="0" layer="20" curve="90"/>
+<wire x1="37" y1="2.54" x2="37" y2="62.46" width="0" layer="20"/>
+<wire x1="37" y1="62.46" x2="34.46" y2="65" width="0" layer="20" curve="90"/>
+<wire x1="34.46" y1="65" x2="2.54" y2="65" width="0" layer="20"/>
+<wire x1="2.54" y1="65" x2="0" y2="62.46" width="0" layer="20" curve="90"/>
+<wire x1="0" y1="62.46" x2="0" y2="2.54" width="0" layer="20"/>
+<wire x1="0" y1="2.54" x2="2.54" y2="0" width="0" layer="20" curve="90"/>
+<text x="6.50875" y="2.2225" size="1.27" layer="25" rot="R180">+5V</text>
+<text x="9.8425" y="6.6675" size="1.27" layer="25" rot="R180">GND</text>
 </plain>
 <attributes>
@@
 </autorouter>
 <elements>
-<element name="C1" library="rcl" package="C0805" value="470n" x="1.5875" y="5.23875" smashed="yes" rot="R270">
-<attribute name="NAME" x="0.9525" y="3.33375" size="1.27" layer="25" rot="R270"/>
-<attribute name="VALUE" x="-0.9525" y="6.50875" size="1.27" layer="27" rot="R270"/>
+<element name="C1" library="rcl" package="C0805" value="470n" x="2.8575" y="5.08" smashed="yes" rot="R270">
+<attribute name="NAME" x="0.47625" y="6.19125" size="1.27" layer="25" rot="R270"/>
+<attribute name="VALUE" x="0.3175" y="6.35" size="1.27" layer="27" rot="R270"/>
 </element>
 <element name="C10" library="rcl" package="C0805" value="100n" x="34.29" y="27.94" smashed="yes" rot="MR180">
@@
 <attribute name="VALUE" x="4.92125" y="59.3725" size="1.27" layer="27" rot="R270"/>
 </element>
-<element name="JP1" library="pinhead" package="1X02SMD" value="" x="6.50875" y="3.4925" smashed="yes">
-<attribute name="VALUE" x="3.96875" y="0.3175" size="1.27" layer="27"/>
+<element name="JP1" library="pinhead" package="1X02SMD" value="" x="6.50875" y="3.81" smashed="yes">
+<attribute name="VALUE" x="3.96875" y="0.635" size="1.27" layer="27"/>
 </element>
 </elements>
@@
 <contactref element="U$1" pad="-"/>
 <polygon width="0.254" layer="1">
-<vertex x="0" y="64.92875"/>
-<vertex x="36.98875" y="64.92875"/>
-<vertex x="36.98875" y="64.77"/>
-<vertex x="36.98875" y="61.43625"/>
-<vertex x="36.98875" y="0"/>
-<vertex x="0" y="0"/>
+<vertex x="36.98875" y="62.38875"/>
+<vertex x="36.98875" y="2.54" curve="-90"/>
+<vertex x="34.44875" y="0"/>
+<vertex x="2.54" y="0" curve="-90"/>
+<vertex x="0" y="2.54"/>
+<vertex x="0" y="62.38875" curve="-90"/>
+<vertex x="2.54" y="64.92875"/>
+<vertex x="34.44875" y="64.92875" curve="-90"/>
 </polygon>
 <polygon width="0.254" layer="16">
-<vertex x="0" y="64.92875"/>
-<vertex x="36.98875" y="64.92875"/>
-<vertex x="36.98875" y="60.48375"/>
-<vertex x="36.98875" y="0"/>
-<vertex x="0" y="0"/>
+<vertex x="36.98875" y="62.38875"/>
+<vertex x="36.98875" y="2.54" curve="-90"/>
+<vertex x="34.44875" y="0"/>
+<vertex x="2.54" y="0" curve="-90"/>
+<vertex x="0" y="2.54"/>
+<vertex x="0" y="62.38875" curve="-90"/>
+<vertex x="2.54" y="64.92875"/>
+<vertex x="34.44875" y="64.92875" curve="-90"/>
 </polygon>
 <wire x1="12.54125" y1="20.6375" x2="14.2875" y2="20.79625" width="0.254" layer="1"/>
@@
 <contactref element="C1" pad="1"/>
 <wire x1="4.1675" y1="16.07375" x2="3.69125" y2="16.11" width="0.4064" layer="1"/>
-<wire x1="1.5875" y1="13.49375" x2="3.69125" y2="15.5975" width="0.4064" layer="1"/>
+<wire x1="1.74625" y1="13.6525" x2="3.69125" y2="15.5975" width="0.4064" layer="1"/>
 <wire x1="3.69125" y1="15.5975" x2="3.69125" y2="16.11" width="0.4064" layer="1"/>
 <contactref element="JP1" pad="1"/>
-<wire x1="1.5875" y1="13.49375" x2="1.5875" y2="6.18875" width="0.4064" layer="1"/>
-<wire x1="1.5875" y1="6.18875" x2="1.59" y2="6.19125" width="0.4064" layer="1"/>
-<wire x1="1.59" y1="6.19125" x2="3.65125" y2="6.19125" width="0.4064" layer="1"/>
-<wire x1="3.65125" y1="6.19125" x2="5.08" y2="4.7625" width="0.4064" layer="1"/>
-<wire x1="5.08" y1="4.7625" x2="5.23875" y2="4.7625" width="0.4064" layer="1"/>
+<wire x1="2.8575" y1="6.03" x2="2.38125" y2="5.55375" width="0.4064" layer="1"/>
+<wire x1="5.3975" y1="5.55375" x2="5.23875" y2="5.08" width="0.4064" layer="1"/>
+<wire x1="2.8575" y1="6.03" x2="5.3975" y2="6.03" width="0.4064" layer="1"/>
+<wire x1="5.3975" y1="6.03" x2="5.23875" y2="5.08" width="0.4064" layer="1"/>
+<wire x1="1.74625" y1="13.6525" x2="1.74625" y2="6.6675" width="0.4064" layer="1"/>
+<wire x1="1.74625" y1="6.6675" x2="2.38375" y2="6.03" width="0.4064" layer="1"/>
+<wire x1="2.38375" y1="6.03" x2="2.8575" y2="6.03" width="0.4064" layer="1"/>
 </signal>
 <signal name="SWCLK">

Commit message: gerber
Parts:
- moved C6 0.16 mm to (35.4, 17.8)
- moved R11 0.16 mm to (32.9, 17.8)
Other:
- outline, holes or cut-outs redrawn
- board text added: "github.com/NicoZellinger/ SensorMonitoring"
- board text added: "universal data aquisition network module v.1.0"
Changed lines of the file:
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@@
 <grid distance="0.00625" unitdist="inch" unit="inch" style="lines" multiple="1" display="no" altdistance="0.025" altunitdist="inch" altunit="inch"/>
 <layers>
-<layer number="1" name="Top" color="4" fill="1" visible="yes" active="yes"/>
-<layer number="16" name="Bottom" color="1" fill="1" visible="yes" active="yes"/>
+<layer number="1" name="Top" color="4" fill="1" visible="no" active="yes"/>
+<layer number="16" name="Bottom" color="1" fill="1" visible="no" active="yes"/>
 <layer number="17" name="Pads" color="2" fill="1" visible="yes" active="yes"/>
 <layer number="18" name="Vias" color="2" fill="1" visible="yes" active="yes"/>
@@
 <wire x1="37" y1="2.54" x2="37" y2="62.46" width="0" layer="20"/>
 <wire x1="37" y1="62.46" x2="34.46" y2="65" width="0" layer="20" curve="90"/>
-<wire x1="34.46" y1="65" x2="2.54" y2="65" width="0" layer="20"/>
-<wire x1="2.54" y1="65" x2="0" y2="62.46" width="0" layer="20" curve="90"/>
+<wire x1="34.46" y1="65" x2="3.175" y2="64.6825" width="0" layer="20"/>
+<wire x1="3.175" y1="64.6825" x2="0" y2="62.46" width="0" layer="20" curve="90"/>
 <wire x1="0" y1="62.46" x2="0" y2="2.54" width="0" layer="20"/>
 <wire x1="0" y1="2.54" x2="2.54" y2="0" width="0" layer="20" curve="90"/>
 <text x="6.50875" y="2.2225" size="1.27" layer="25" rot="R180">+5V</text>
 <text x="9.8425" y="6.6675" size="1.27" layer="25" rot="R180">GND</text>
+<text x="5.23875" y="35.40125" size="1.778" layer="25" rot="R90">universal data aquisition
+ network module v.1.0</text>
+<text x="34.13125" y="40.3225" size="1.4224" layer="25" rot="R90">github.com/NicoZellinger/
+SensorMonitoring</text>
 </plain>
 <attributes>
@@
 <attribute name="VALUE" x="31.75" y="9.8425" size="1.27" layer="28" rot="MR0"/>
 </element>
-<element name="C6" library="rcl" package="C0805" value="20p" x="35.56" y="17.78" smashed="yes" rot="R90">
-<attribute name="NAME" x="34.76625" y="15.71625" size="1.27" layer="25" rot="R270"/>
-<attribute name="VALUE" x="38.1" y="16.51" size="1.27" layer="27" rot="R90"/>
+<element name="C6" library="rcl" package="C0805" value="20p" x="35.40125" y="17.78" smashed="yes" rot="R90">
+<attribute name="NAME" x="34.6075" y="15.71625" size="1.27" layer="25" rot="R270"/>
+<attribute name="VALUE" x="37.94125" y="16.51" size="1.27" layer="27" rot="R90"/>
 </element>
 <element name="C7" library="rcl" package="C0805" value="100n" x="30.48" y="9.525" smashed="yes" rot="MR0">
@@
 <attribute name="VALUE" x="3.175" y="25.4" size="1.27" layer="28" rot="MR0"/>
 </element>
-<element name="R11" library="rcl" package="R0805" value="390" x="32.7025" y="17.78" smashed="yes" rot="R90">
-<attribute name="NAME" x="31.90875" y="15.71625" size="1.27" layer="25" rot="R270"/>
-<attribute name="VALUE" x="35.2425" y="17.145" size="1.27" layer="27" rot="R90"/>
+<element name="R11" library="rcl" package="R0805" value="390" x="32.86125" y="17.78" smashed="yes" rot="R90">
+<attribute name="NAME" x="32.0675" y="15.71625" size="1.27" layer="25" rot="R270"/>
+<attribute name="VALUE" x="35.40125" y="17.145" size="1.27" layer="27" rot="R90"/>
 </element>
 <element name="R12" library="rcl" package="R0805" value="10k" x="2.54" y="22.86" smashed="yes" rot="MR0">
@@
 <element name="U$5" library="breakout_base" package="BREAKOUT_FOOTPRINT_V1" value="BREAKOUT_FP_V1" x="33.655" y="63.1825" rot="MR270"/>
 <element name="R4" library="rcl" package="R0805" value="10k" x="7.46125" y="58.7375" smashed="yes" rot="R270">
-<attribute name="NAME" x="4.92125" y="59.84875" size="1.27" layer="25" rot="R270"/>
+<attribute name="NAME" x="8.255" y="60.6425" size="1.27" layer="25" rot="R90"/>
 <attribute name="VALUE" x="4.92125" y="59.3725" size="1.27" layer="27" rot="R270"/>
 </element>
@@
 <wire x1="34.13125" y1="22.7965" x2="34.13125" y2="18.7325" width="0.254" layer="1"/>
 <wire x1="34.13125" y1="18.7325" x2="34.13375" y2="18.73" width="0.254" layer="1"/>
-<wire x1="34.13375" y1="18.73" x2="35.56" y2="18.73" width="0.254" layer="1"/>
-<wire x1="32.7025" y1="18.73" x2="34.13375" y2="18.73" width="0.254" layer="1"/>
+<wire x1="34.13375" y1="18.73" x2="35.40125" y2="18.73" width="0.254" layer="1"/>
+<wire x1="32.86125" y1="18.73" x2="34.13375" y2="18.73" width="0.254" layer="1"/>
 </signal>
 <signal name="OSC_IN">
@@
 <wire x1="31.90875" y1="16.8275" x2="32.385" y2="16.8275" width="0.254" layer="1"/>
 <wire x1="32.385" y1="16.8275" x2="32.7025" y2="16.8275" width="0.254" layer="1"/>
-<wire x1="32.7025" y1="16.83" x2="32.3875" y2="16.83" width="0.254" layer="1"/>
+<wire x1="32.86125" y1="16.83" x2="32.3875" y2="16.83" width="0.254" layer="1"/>
 <wire x1="32.3875" y1="16.83" x2="32.385" y2="16.8275" width="0.254" layer="1"/>
 </signal>
@@
 </board>
 </drawing>
+<compatibility>
+<note version="6.3" minversion="6.2.2" severity="warning">
+Since Version 6.2.2 text objects can contain more than one line,
+which will not be processed correctly with this version.
+</note>
+</compatibility>
 </eagle>
