File: SensorPCB/SensorPCB.sch (EAGLE design)
At the start: 32 parts, among them T1 33u

Commit message: delet temp sensor + route all signal wires
Parts:
- removed MCP9808: MCP9808-E/MS, mcp9808:MCP9808-E/MS
Connections:
- removed net ALERT: MCP9808.ALERT
- net +3V3: no longer MCP9808.VDD
- net GND: no longer MCP9808.A0, MCP9808.A1, MCP9808.A2, MCP9808.GND
- net I2C1_SCL_SENSOR: no longer MCP9808.SCL
- net I2C1_SDA_SENSOR: no longer MCP9808.SDA
Other:
- note removed: "Default Sensor MCP9808 Microchip Temp. Sensor"
- note removed: "I2C address 0011000"
- note removed: "Second Default Sensor?"
- moved on the sheet: C3, C5, C7, C8, IRF7301_SENSOR, IRF7301_WLAN, R1, R10, R2, R3, R6, R9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

Commit message: edit tname and bname
Parts:
- renumbered IRF7301_SENSOR to IRF7301_S, IRF7301_WLAN to IRF7301_W
Changed lines of the file:
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@@
 <attribute name="WEBSITE" value="http://www.reichelt.de/LM-3940-IS3-3/3/index.html?&amp;ACTION=3&amp;LA=446&amp;ARTICLE=109408&amp;artnr=LM+3940+IS3%2C3&amp;SEARCH=SPANNUNGsregler+3%2C3v"/>
 </part>
-<part name="IRF7301_WLAN" library="irf7301_symb" deviceset="IRF7301" device=""/>
+<part name="IRF7301_W" library="irf7301_symb" deviceset="IRF7301" device=""/>
 <part name="SUPPLY1" library="supply2" deviceset="GND" device=""/>
 <part name="SUPPLY6" library="supply2" deviceset="GND" device=""/>
-<part name="IRF7301_SENSOR" library="irf7301_symb" deviceset="IRF7301" device=""/>
+<part name="IRF7301_S" library="irf7301_symb" deviceset="IRF7301" device=""/>
 <part name="SUPPLY7" library="supply2" deviceset="GND" device=""/>
 <part name="SUPPLY8" library="supply2" deviceset="GND" device=""/>
@@
 <attribute name="WEBSITE" x="81.28" y="228.6" size="1.778" layer="96" display="off"/>
 </instance>
-<instance part="IRF7301_WLAN" gate="G$1" x="238.76" y="109.22"/>
+<instance part="IRF7301_W" gate="G$1" x="238.76" y="109.22"/>
 <instance part="SUPPLY1" gate="GND" x="210.82" y="116.84" rot="R270"/>
 <instance part="SUPPLY6" gate="GND" x="210.82" y="106.68" rot="R270"/>
-<instance part="IRF7301_SENSOR" gate="G$1" x="238.76" y="63.5"/>
+<instance part="IRF7301_S" gate="G$1" x="238.76" y="63.5"/>
 <instance part="SUPPLY7" gate="GND" x="208.28" y="71.12" rot="R270"/>
 <instance part="SUPPLY8" gate="GND" x="208.28" y="60.96" rot="R270"/>
@@
 </segment>
 <segment>
-<pinref part="IRF7301_WLAN" gate="G$1" pin="S1"/>
+<pinref part="IRF7301_W" gate="G$1" pin="S1"/>
 <pinref part="SUPPLY1" gate="GND" pin="GND"/>
 <wire x1="226.06" y1="116.84" x2="213.36" y2="116.84" width="0.1524" layer="91"/>
@@
 <segment>
 <pinref part="SUPPLY6" gate="GND" pin="GND"/>
-<pinref part="IRF7301_WLAN" gate="G$1" pin="S2"/>
+<pinref part="IRF7301_W" gate="G$1" pin="S2"/>
 <wire x1="213.36" y1="106.68" x2="226.06" y2="106.68" width="0.1524" layer="91"/>
 </segment>
 <segment>
-<pinref part="IRF7301_SENSOR" gate="G$1" pin="S1"/>
+<pinref part="IRF7301_S" gate="G$1" pin="S1"/>
 <pinref part="SUPPLY7" gate="GND" pin="GND"/>
 <wire x1="226.06" y1="71.12" x2="210.82" y2="71.12" width="0.1524" layer="91"/>
@@
 <segment>
 <pinref part="SUPPLY8" gate="GND" pin="GND"/>
-<pinref part="IRF7301_SENSOR" gate="G$1" pin="S2"/>
+<pinref part="IRF7301_S" gate="G$1" pin="S2"/>
 <wire x1="210.82" y1="60.96" x2="226.06" y2="60.96" width="0.1524" layer="91"/>
 </segment>
@@
 <net name="GND_WLAN" class="0">
 <segment>
-<pinref part="IRF7301_WLAN" gate="G$1" pin="D1"/>
+<pinref part="IRF7301_W" gate="G$1" pin="D1"/>
 <wire x1="251.46" y1="114.3" x2="271.78" y2="114.3" width="0.1524" layer="91"/>
 <label x="259.08" y="114.3" size="1.778" layer="95"/>
 </segment>
 <segment>
-<pinref part="IRF7301_WLAN" gate="G$1" pin="D2"/>
+<pinref part="IRF7301_W" gate="G$1" pin="D2"/>
 <wire x1="271.78" y1="104.14" x2="251.46" y2="104.14" width="0.1524" layer="91"/>
 <label x="259.08" y="104.14" size="1.778" layer="95"/>
@@
 <net name="GND_SENSOR" class="0">
 <segment>
-<pinref part="IRF7301_SENSOR" gate="G$1" pin="D1"/>
+<pinref part="IRF7301_S" gate="G$1" pin="D1"/>
 <wire x1="251.46" y1="68.58" x2="274.32" y2="68.58" width="0.1524" layer="91"/>
 <label x="259.08" y="68.58" size="1.778" layer="95"/>
 </segment>
 <segment>
-<pinref part="IRF7301_SENSOR" gate="G$1" pin="D2"/>
+<pinref part="IRF7301_S" gate="G$1" pin="D2"/>
 <wire x1="274.32" y1="58.42" x2="251.46" y2="58.42" width="0.1524" layer="91"/>
 <label x="259.08" y="58.42" size="1.778" layer="95"/>
@@
 </segment>
 <segment>
-<pinref part="IRF7301_WLAN" gate="G$1" pin="G1"/>
+<pinref part="IRF7301_W" gate="G$1" pin="G1"/>
 <wire x1="226.06" y1="111.76" x2="208.28" y2="111.76" width="0.1524" layer="91"/>
 <label x="210.82" y="111.76" size="1.778" layer="95"/>
 </segment>
 <segment>
-<pinref part="IRF7301_WLAN" gate="G$1" pin="G2"/>
+<pinref part="IRF7301_W" gate="G$1" pin="G2"/>
 <wire x1="226.06" y1="101.6" x2="208.28" y2="101.6" width="0.1524" layer="91"/>
 <label x="210.82" y="101.6" size="1.778" layer="95"/>
@@
 </segment>
 <segment>
-<pinref part="IRF7301_SENSOR" gate="G$1" pin="G2"/>
+<pinref part="IRF7301_S" gate="G$1" pin="G2"/>
 <wire x1="226.06" y1="55.88" x2="205.74" y2="55.88" width="0.1524" layer="91"/>
 <label x="205.74" y="55.88" size="1.778" layer="95"/>
 </segment>
 <segment>
-<pinref part="IRF7301_SENSOR" gate="G$1" pin="G1"/>
+<pinref part="IRF7301_S" gate="G$1" pin="G1"/>
 <wire x1="226.06" y1="66.04" x2="205.74" y2="66.04" width="0.1524" layer="91"/>
 <label x="205.74" y="66.04" size="1.778" layer="95"/>

Commit message: closed #1
Parts:
- removed U$2: 5V_POWER_SUPPLY, 5V_POWER_SUPPLY:5V_POWER_SUPPLY
- added JP1: (no value), pinhead:PINHD-1X2_2.54-SMD
Connections:
- net +5V: now also JP1.1; no longer U$2.-
- net GND: now also JP1.2; no longer U$2.+
Changed lines of the file:
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@@
 <part name="+3V15" library="supply1" deviceset="+3V3" device=""/>
 <part name="SUPPLY24" library="supply2" deviceset="GND" device=""/>
-<part name="U$2" library="5V_POWER_SUPPLY" deviceset="5V_POWER_SUPPLY" device=""/>
 <part name="P+2" library="supply1" deviceset="+5V" device=""/>
 <part name="SUPPLY25" library="supply2" deviceset="GND" device=""/>
 <part name="R4" library="rcl" deviceset="R-EU_" device="R0805" value="10k"/>
 <part name="+3V7" library="supply1" deviceset="+3V3" device=""/>
+<part name="JP1" library="pinhead" deviceset="PINHD-1X2" device="_2.54-SMD"/>
 </parts>
 <sheets>
@@
 <instance part="+3V15" gate="G$1" x="43.18" y="185.42"/>
 <instance part="SUPPLY24" gate="GND" x="17.78" y="172.72"/>
-<instance part="U$2" gate="G$1" x="30.48" y="223.52"/>
-<instance part="P+2" gate="1" x="43.18" y="231.14"/>
+<instance part="P+2" gate="1" x="43.18" y="233.68"/>
 <instance part="SUPPLY25" gate="GND" x="17.78" y="218.44"/>
 <instance part="R4" gate="G$1" x="294.64" y="223.52" rot="R180"/>
 <instance part="+3V7" gate="G$1" x="287.02" y="223.52" rot="R90"/>
+<instance part="JP1" gate="G$1" x="33.02" y="223.52"/>
 </instances>
 <busses>
@@
 <pinref part="SUPPLY25" gate="GND" pin="GND"/>
 <wire x1="17.78" y1="220.98" x2="17.78" y2="223.52" width="0.1524" layer="91"/>
-<pinref part="U$2" gate="G$1" pin="+"/>
-<wire x1="17.78" y1="223.52" x2="20.32" y2="223.52" width="0.1524" layer="91"/>
+<pinref part="JP1" gate="G$1" pin="2"/>
+<wire x1="17.78" y1="223.52" x2="30.48" y2="223.52" width="0.1524" layer="91"/>
 </segment>
 </net>
@@
 </segment>
 <segment>
-<pinref part="U$2" gate="G$1" pin="-"/>
 <pinref part="P+2" gate="1" pin="+5V"/>
-<wire x1="40.64" y1="223.52" x2="43.18" y2="223.52" width="0.1524" layer="91"/>
-<wire x1="43.18" y1="223.52" x2="43.18" y2="228.6" width="0.1524" layer="91"/>
+<pinref part="JP1" gate="G$1" pin="1"/>
+<wire x1="43.18" y1="226.06" x2="43.18" y2="231.14" width="0.1524" layer="91"/>
+<wire x1="30.48" y1="226.06" x2="43.18" y2="226.06" width="0.1524" layer="91"/>
 </segment>
 </net>

Commit message: some last improvements to get ready for version 1.0
Parts:
- renumbered QUARZ-HC49 to QUARZ
Changed lines of the file:
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@@
 <part name="+3V6" library="supply1" deviceset="+3V3" device=""/>
 <part name="SUPPLY11" library="supply2" deviceset="GND" device=""/>
-<part name="QUARZ-HC49" library="quarz_hc49_smd" deviceset="QUARZ_HC49-SMD" device=""/>
+<part name="QUARZ" library="quarz_hc49_smd" deviceset="QUARZ_HC49-SMD" device=""/>
 <part name="SUPPLY10" library="supply2" deviceset="GND" device=""/>
 <part name="SUPPLY12" library="supply2" deviceset="GND" device=""/>
@@
 <instance part="+3V6" gate="G$1" x="109.22" y="10.16" rot="R180"/>
 <instance part="SUPPLY11" gate="GND" x="104.14" y="12.7"/>
-<instance part="QUARZ-HC49" gate="G$1" x="27.94" y="68.58" rot="R90"/>
+<instance part="QUARZ" gate="G$1" x="27.94" y="68.58" rot="R90"/>
 <instance part="SUPPLY10" gate="GND" x="10.16" y="66.04" rot="R270"/>
 <instance part="SUPPLY12" gate="GND" x="10.16" y="71.12" rot="R270"/>
@@
 <net name="N$4" class="0">
 <segment>
-<pinref part="QUARZ-HC49" gate="G$1" pin="1"/>
+<pinref part="QUARZ" gate="G$1" pin="1"/>
 <junction x="27.94" y="66.04"/>
 <wire x1="27.94" y1="66.04" x2="22.86" y2="66.04" width="0.1524" layer="91"/>
@@
 <net name="OSC_IN" class="0">
 <segment>
-<pinref part="QUARZ-HC49" gate="G$1" pin="2"/>
+<pinref part="QUARZ" gate="G$1" pin="2"/>
 <pinref part="STM32L051C8T6" gate="G$1" pin="OSC_IN"/>
 <wire x1="43.18" y1="71.12" x2="27.94" y2="71.12" width="0.1524" layer="91"/>
