File: SensorPCB/gerber/SensorPCB.brd (EAGLE design)
At the start: 37 x 65 mm, 31 parts, among them T1 33u

Commit message: some last improvements to get ready for version 1.0
Parts:
- renumbered QUARZ-HC49 to QUARZ
Routing:
- net PA7: track 28.2 -> 26.6 mm
- net PA6: track 31.1 -> 29.7 mm
- net PA5: track 34.1 -> 32.9 mm
- net PA4: track 37.0 -> 36.0 mm
- net USART2_RX_SENSOR: track 62.7 -> 61.9 mm
- net N$1: track 18.9 -> 19.6 mm
Other:
- board text added: "+3V3"
- board text added: "RX"
- board text added: "SWCLK"
- board text added: "SWDIO"
- board text added: "TX"
